Commit message: 05/02 updates on gazebo, xacro, new launch file and extension to the launch file

File: robot.xacro (robot description, xacro)
@@ -2,5 +2,5 @@
 <robot  name="differential_drive_robot" xmlns:xacro="http://www.ros.org/wiki/xacro" >
 <!-- Body properties-->
-<xacro:property name='body_link_x_dim' value='1'/>
+<xacro:property name='body_link_x_dim' value='1.0'/>
 <xacro:property name='body_link_y_dim' value='0.6'/>
 <xacro:property name='body_link_z_dim' value='0.3'/>
@@ -20,28 +20,28 @@
 <xacro:property name='body_mass' value='${body_density*body_link_x_dim*body_link_y_dim*body_link_z_dim}'/>
 <xacro:property name='wheel_mass' value='${wheel_density*pi_const*wheel_link_radius*wheel_link_radius*wheel_link_length}'/>
-<xacro:property name='caster_mass' value='${caster_density*(4.0/3.0)*pi_const*caster_link_radius*caster_link_radius}'/>
+<xacro:property name='caster_mass' value='${caster_density*(4.0/3.0)*pi_const*caster_link_radius*caster_link_radius*caster_link_radius}'/>
 <!--Moment of inertia-->
 <xacro:property name='Iz_wheel' value='${0.5*wheel_mass*wheel_link_radius*wheel_link_radius}'/>
 <xacro:property name='I_wheel' value='${1.0/12.0*wheel_mass*(3.0*wheel_link_radius*wheel_link_radius+wheel_link_length*wheel_link_length)}'/>
-<xacro:property name='Iz_wheel' value='${(2.0/5.0)*caster_mass*caster_link_radius*caster_link_radius}'/>
+<xacro:property name='I_caster' value='${(2.0/5.0)*caster_mass*caster_link_radius*caster_link_radius}'/>
 <xacro:macro name='inertia_wheel'>
     <inertial>
-    <origin rpy='0 0 0' xyz='0 0 0'>
-    <mass value="${wheel_mass}">
-    <inertia ixx='${I_wheel}' ixy='0.0' ixz='0.0' iyy='${I_wheel}' iyz='0' izz='${Iz_wheel}'/>
+	    <origin rpy='0 0 0' xyz='0 0 0'/>
+	    <mass value="${wheel_mass}"/>
+	    <inertia ixx='${I_wheel}' ixy='0.0' ixz='0.0' iyy='${I_wheel}' iyz='0' izz='${Iz_wheel}'/>
     </inertial>
 </xacro:macro>
 <xacro:macro name='inertia_caster'>
     <inertial>
-    <origin rpy='0 0 0' xyz='0 0 0'>
-    <mass value="${caster_mass}">
-    <inertia ixx='${I_caster}' ixy='0.0' ixz='0.0' iyy='${I_caster}' iyz='0' izz='${Iz_caster}'/>
+	    <origin rpy='0 0 0' xyz='0 0 0'/>
+	    <mass value="${caster_mass}"/>
+	    <inertia ixx='${I_caster}' ixy='0.0' ixz='0.0' iyy='${I_caster}' iyz='0' izz='${I_caster}'/>
     </inertial>
 </xacro:macro>
 <xacro:include filename='$(find driverless_robot)/model/robot.gazebo' />
-<link name='dummy'>
+<link name='base_link'>
 </link>
-<joint name='dummy_joint' type='fixed'>
-    <parent link='dummy'/>
+<joint name='base_joint' type='fixed'>
+    <parent link='base_link'/>
     <child link='body_link'/>
 </joint>
@@ -57,24 +57,23 @@
             <box size='${body_link_x_dim} ${body_link_y_dim} ${body_link_z_dim}'/>
         </geometry>
-        <origin rpy='0 0 0' xyz='0 0 0'/>
+       <origin rpy='0 0 0' xyz='0 0 0'/>
     </collision>
     <inertial>
         <origin rpy='0 0 0' xyz='0 0 0'/>
         <mass value="${body_mass}"/>
-    <inertia ixx='${(1/12)*body_mass*(body_link_y_dim*body_link_y_dim+body_link_z_dim*body_link_z_dim)}' ixy="0"
-    izz='${(1/12)*body_mass*(body_link_y_dim*body_link_y_dim+body_link_x_dim*body_link_x_dim)}'/>
+    	<inertia ixx='${(1.0/12.0)*body_mass*(body_link_y_dim*body_link_y_dim+body_link_z_dim*body_link_z_dim)}' ixy="0" ixz='0' iyy='${(1.0/12.0)*body_mass*(body_link_x_dim*body_link_x_dim+body_link_z_dim*body_link_z_dim)}' iyz='0' izz='${(1.0/12.0)*body_mass*(body_link_y_dim*body_link_y_dim+body_link_x_dim*body_link_x_dim)}'/>
     </inertial>
 </link>
 <joint name='wheel1_joint' type='continuous'>
-    <parent link='body_link'/>
+    <parent link='base_link'/>
     <child link='wheel1_link'/>
-    <origin xyz='${-2*wheel_link_radius} ${-body_link_y_dim/2-wheel_link_length/2} ${wheel_link_z_location} ' rpy='0 0 0' />
+    <origin xyz='-${2*wheel_link_radius} -${(body_link_y_dim/2)-(wheel_link_length/2)} ${wheel_link_z_location} ' rpy='0 0 0' />
     <axis xyz='0 1 0'/>
-    <limit effor='1000' velocity='1000'/>
-    <dynamics damping='1.0' fricition='1.0'>
+    <limit effort='1000' velocity='1000'/>
+    <dynamics damping='1.0' fricition='1.0'/>
 </joint>
 <link name='wheel1_link'>
     <visual>
-    <origin rpy='1.570795 0 0' xyz='0 0 0'/>
+    	<origin rpy='1.570795 0 0' xyz='0 0 0'/>
         <geometry>
             <cylinder length='${wheel_link_length}' radius='${wheel_link_radius}'/>
@@ -87,13 +86,13 @@
         </geometry>
     </collision>
-    <xacro:inertial_wheel/>
+    <xacro:inertia_wheel/>
 </link>
 <joint name='wheel2_joint' type='continuous'>
     <parent link='body_link'/>
     <child link='wheel2_link'/>
-    <origin xyz='${-2*wheel_link_radius} ${body_link_y_dim/2+wheel_link_length/2} ${wheel_link_z_location} ' rpy='0 0 0' />
+    <origin xyz='-${2*wheel_link_radius} ${body_link_y_dim/2+wheel_link_length/2} ${wheel_link_z_location} ' rpy='0 0 0' />
     <axis xyz='0 1 0'/>
-    <limit effor='1000' velocity='1000'/>
-    <dynamics damping='1.0' fricition='1.0'>
+    <limit effort='1000' velocity='1000'/>
+    <dynamics damping='1.0' fricition='1.0'/>
 </joint>
 <link name='wheel2_link'>
@@ -110,9 +109,9 @@
         </geometry>
     </collision>
-    <xacro:inertial_wheel/>
+    <xacro:inertia_wheel/>
 </link>
 <joint name='caster_joint' type='fixed'>
-    <parent link='caster_link'/>
-    <child link='body_link'/>
+    <parent link='body_link'/>
+    <child link='caster_link'/>
     <origin xyz='${2*caster_link_radius} 0 ${caster_link_z_location}' rpy='0 0 0'/>
 </joint>
@@ -130,5 +129,5 @@
         </geometry>
     </collision>
-    <xacro:inertial_caster />
+    <xacro:inertia_caster/>
 </link>
 </robot>

Commit message: up-to-date files HARD 07/02

File: robot.xacro (robot description, xacro)
@@ -11,18 +11,29 @@
 <xacro:property name='caster_link_radius' value='0.15'/>
 <xacro:property name='caster_link_z_location' value='-0.1'/>
+<!-- Lidar properties-->
+<xacro:property name='lidar_link_radius' value='0.05'/>
+<xacro:property name='lidar_link_length' value='0.04'/>
+<xacro:property name='lidar_link_z_location' value='0.16'/>
 <!-- Material properties-->
 <xacro:property name='body_density' value='2710.0'/>
 <xacro:property name='wheel_density' value='2710.0'/>
 <xacro:property name='caster_density' value='2710.0'/>
+<xacro:property name='lidar_density' value='1600.0'/>
 <!--Pi const-->
 <xacro:property name='pi_const' value='3.14159265'/>
-<!--Robot body mass, wheel mass, caster mass-->
+<!--Robot body mass, wheel mass, caster mass, lidar mass-->
 <xacro:property name='body_mass' value='${body_density*body_link_x_dim*body_link_y_dim*body_link_z_dim}'/>
 <xacro:property name='wheel_mass' value='${wheel_density*pi_const*wheel_link_radius*wheel_link_radius*wheel_link_length}'/>
 <xacro:property name='caster_mass' value='${caster_density*(4.0/3.0)*pi_const*caster_link_radius*caster_link_radius*caster_link_radius}'/>
+<xacro:property name='lidar_mass' value='${lidar_density*pi_const*lidar_link_radius*lidar_link_radius*lidar_link_length}'/>
 <!--Moment of inertia-->
+<!--Moment of inertia wheel-->
 <xacro:property name='Iz_wheel' value='${0.5*wheel_mass*wheel_link_radius*wheel_link_radius}'/>
 <xacro:property name='I_wheel' value='${1.0/12.0*wheel_mass*(3.0*wheel_link_radius*wheel_link_radius+wheel_link_length*wheel_link_length)}'/>
+<!--Moment of caster wheel-->
 <xacro:property name='I_caster' value='${(2.0/5.0)*caster_mass*caster_link_radius*caster_link_radius}'/>
+<!--Moment of lidar-->
+<xacro:property name='Iz_lidar' value='${0.5*lidar_mass*lidar_link_radius*lidar_link_radius}'/>
+<xacro:property name='I_lidar' value='${1.0/12.0*lidar_mass*(3.0*lidar_link_radius*lidar_link_radius+lidar_link_length*lidar_link_length)}'/>
 <xacro:macro name='inertia_wheel'>
     <inertial>
@@ -37,4 +48,11 @@
 	    <mass value="${caster_mass}"/>
 	    <inertia ixx='${I_caster}' ixy='0.0' ixz='0.0' iyy='${I_caster}' iyz='0' izz='${I_caster}'/>
+    </inertial>
+</xacro:macro>
+<xacro:macro name='inertia_lidar'>
+    <inertial>
+        <origin rpy='0 0 0' xyz='0 0 0'/>
+        <mass value="${lidar_mass}"/>
+        <inertia ixx='${I_lidar}' ixy='0.0' ixz='0.0' iyy='${I_lidar}' iyz='0' izz='${Iz_lidar}'/>
     </inertial>
 </xacro:macro>
@@ -65,8 +83,9 @@
     </inertial>
 </link>
+<!-- Wheel 1 joint and link-->
 <joint name='wheel1_joint' type='continuous'>
     <parent link='base_link'/>
     <child link='wheel1_link'/>
-    <origin xyz='-${2*wheel_link_radius} -${(body_link_y_dim/2)-(wheel_link_length/2)} ${wheel_link_z_location} ' rpy='0 0 0' />
+    <origin xyz='-${2*wheel_link_radius} ${-(body_link_y_dim/2)-(wheel_link_length/2)} ${wheel_link_z_location} ' rpy='0 0 0' />
     <axis xyz='0 1 0'/>
     <limit effort='1000' velocity='1000'/>
@@ -88,8 +107,9 @@
     <xacro:inertia_wheel/>
 </link>
+<!-- Wheel 2 joint and link-->
 <joint name='wheel2_joint' type='continuous'>
     <parent link='body_link'/>
     <child link='wheel2_link'/>
-    <origin xyz='-${2*wheel_link_radius} ${body_link_y_dim/2+wheel_link_length/2} ${wheel_link_z_location} ' rpy='0 0 0' />
+    <origin xyz='-${2*wheel_link_radius} ${(body_link_y_dim/2)+(wheel_link_length/2)} ${wheel_link_z_location} ' rpy='0 0 0' />
     <axis xyz='0 1 0'/>
     <limit effort='1000' velocity='1000'/>
@@ -111,4 +131,5 @@
     <xacro:inertia_wheel/>
 </link>
+<!-- Caster joint and link-->
 <joint name='caster_joint' type='fixed'>
     <parent link='body_link'/>
@@ -131,3 +152,22 @@
     <xacro:inertia_caster/>
 </link>
+<!-- Lidar joint and link-->
+<joint name="lidar_joint" type='fixed'>
+    <parent link='body_link'/>
+    <child link='lidar_link'/>
+    <origin xyz='0.1 0 ${lidar_link_z_location}' rpy='0 0 0'/>
+</joint>
+<link name='lidar_link'>
+    <visual>
+        <geometry>
+            <cylinder radius='${lidar_link_radius}' length='${lidar_link_length}'/>
+        </geometry>
+    </visual>
+    <collision>
+        <geometry>
+            <cylinder radius='${lidar_link_radius}' length='${lidar_link_length}'/>
+        </geometry>
+    </collision>
+    <xacro:inertia_lidar/>
+</link>
 </robot>
